File: mk19-pcb.kicad_pcb (KiCad board)
At the start: 2 copper layers, 0 parts

Commit message: all new features added, fixes implemented, ready to start arranging and routing
Parts:
- added 5WAY1: Conn_01x08_Socket, Connector_JST:JST_EH_S8B-EH_1x08_P2.50mm_Horizontal, F.Cu at (65.6, 136.0)
- added ADC1: Conn_01x03_Socket, Connector_JST:JST_EH_B3B-EH-A_1x03_P2.50mm_Vertical, F.Cu at (176.2, 25.1)
- added AUDIO1: Conn_01x03_Socket, Connector_JST:JST_EH_B3B-EH-A_1x03_P2.50mm_Vertical, F.Cu at (204.6, 65.6)
- added C1: 100nF, ct-kicad:C0402, F.Cu at (123.8, 121.5)
- added C10: CL31B105KBHNNNE, ct-kicad:C1206, F.Cu at (185.7, 123.6)
- added C11: CL31B105KBHNNNE, ct-kicad:C1206, F.Cu at (165.7, 123.5)
- added C12: CL31B105KBHNNNE, ct-kicad:C1206, F.Cu at (175.3, 123.4)
- added C2: 100nF, ct-kicad:C0402, F.Cu at (123.8, 94.5)
- added C3: 100nF, ct-kicad:C0402, F.Cu at (123.8, 109.5)
- added C4: 100nF, ct-kicad:C0402, F.Cu at (123.8, 74.5)
- added C5: 100nF, ct-kicad:C0402, F.Cu at (161.4, 65.6)
- added C6: 100nF, ct-kicad:C0402, F.Cu at (164.3, 67.6)
- added C7: CL31B105KBHNNNE, ct-kicad:C1206, F.Cu at (120.1, 30.7)
- added C8: CL31B105KBHNNNE, ct-kicad:C1206, F.Cu at (133.9, 29.4)
- added C9: CL31B105KBHNNNE, ct-kicad:C1206, F.Cu at (126.9, 29.1)
- added COL1: Conn_01x08_Socket, Connector_JST:JST_EH_S8B-EH_1x08_P2.50mm_Horizontal, F.Cu at (66.2, 72.3)
- added COL2: Conn_01x08_Socket, Connector_JST:JST_EH_S8B-EH_1x08_P2.50mm_Horizontal, F.Cu at (48.7, 68.1)
- added COL_CS_MOS1: 2N7002, ct-kicad:SOT-23-3_L2.9-W1.3-P1.90-LS2.4-BR, F.Cu at (123.8, 86.5)
- added COL_JOIN1: Conn_01x02_Socket, Connector_PinSocket_2.54mm:PinSocket_1x02_P2.54mm_Vertical, F.Cu at (124.6, 79.6)
- added COL_JOIN2: Conn_01x02_Socket, Connector_PinSocket_2.54mm:PinSocket_1x02_P2.54mm_Vertical, F.Cu at (130.5, 107.8)
- added COL_JOIN3: Conn_01x02_Socket, Connector_PinSocket_2.54mm:PinSocket_1x02_P2.54mm_Vertical, F.Cu at (133.4, 116.2)
- added CYBOARD-MACRO1: HC-FPC-05-10-16RLTAG, ct-kicad:FPC-SMD_16P-P0.50_HCTL_HC-FPC-05-10-16RLTAG, F.Cu at (142.0, 173.7)
- added CYBOARD-MAIN1: ECT818001569, ct-kicad:FPC-SMD_ECT818001569, F.Cu at (153.0, 173.7)
- added D1: SMF5_0CA_C364279, ct-kicad:SOD-123FL_L2.8-W1.8-LS3.7-BI, F.Cu at (168.3, 59.4)
- added DBG1: Conn_01x03_Socket, Connector_JST:JST_EH_B3B-EH-A_1x03_P2.50mm_Vertical, F.Cu at (197.8, 118.2)
- added F1: MF-NSMF075-2, ct-kicad:F1206, F.Cu at (170.8, 59.3)
- added FAL1: Conn_01x08_Socket, Connector_JST:JST_EH_S8B-EH_1x08_P2.50mm_Horizontal, F.Cu at (202.9, 80.2)
- added FAL2: Conn_01x08_Socket, Connector_JST:JST_EH_S8B-EH_1x08_P2.50mm_Horizontal, F.Cu at (202.9, 105.2)
- added FAL_PINS1: Conn_01x04_Socket, Connector_PinSocket_2.54mm:PinSocket_1x04_P2.54mm_Vertical, F.Cu at (199.1, 95.0)
- added G2: Conn_01x01_Socket, Connector_Pin:Pin_D1.0mm_L10.0mm, F.Cu at (233.5, 127.0)
- added G3: Conn_01x01_Socket, Connector_Pin:Pin_D1.0mm_L10.0mm, F.Cu at (233.5, 131.0)
- added G6: Conn_01x01_Socket, Connector_Pin:Pin_D1.0mm_L10.0mm, F.Cu at (237.5, 131.0)
- added H1: MountingHole, MountingHole:MountingHole_3.2mm_M3_Pad_Via, F.Cu at (85.0, 55.0)
- added H2: MountingHole, MountingHole:MountingHole_3.2mm_M3_Pad_Via, F.Cu at (205.0, 55.0)
- added H3: MountingHole, MountingHole:MountingHole_3.2mm_M3_Pad_Via, F.Cu at (85.0, 130.0)
- added H4: MountingHole, MountingHole:MountingHole_3.2mm_M3_Pad_Via, F.Cu at (205.0, 130.0)
- added J10: Conn_01x02_Socket, Connector_PinSocket_2.54mm:PinSocket_1x02_P2.54mm_Vertical, F.Cu at (231.0, 89.4)
- added J11: Conn_01x02_Socket, Connector_PinSocket_2.54mm:PinSocket_1x02_P2.54mm_Vertical, F.Cu at (194.2, 64.1)
- added J12: Conn_01x02_Socket, Connector_PinSocket_2.54mm:PinSocket_1x02_P2.54mm_Vertical, F.Cu at (196.6, 68.0)
- added J4: Conn_01x02_Socket, Connector_PinSocket_2.54mm:PinSocket_1x02_P2.54mm_Vertical, F.Cu at (226.6, 89.4)
- added J5: Conn_01x02_Socket, Connector_JST:JST_EH_B2B-EH-A_1x02_P2.50mm_Vertical, F.Cu at (120.7, 23.9)
- added J6: Conn_01x02_Socket, Connector_JST:JST_EH_B2B-EH-A_1x02_P2.50mm_Vertical, F.Cu at (126.9, 24.0)
- added J7: Conn_01x02_Socket, Connector_JST:JST_EH_B2B-EH-A_1x02_P2.50mm_Vertical, F.Cu at (133.2, 23.9)
- added J9: Conn_01x02_Socket, Connector_PinSocket_2.54mm:PinSocket_1x02_P2.54mm_Vertical, F.Cu at (221.9, 89.4)
- added L1: MPZ2012S101AT000, ct-kicad:L0805, F.Cu at (171.8, 63.0)
- added LED-LVL1: SN74LVC1T45DRL, ct-kicad:SOT-563_L1.6-W1.2-P0.50-LS1.6-BR, F.Cu at (161.4, 68.1)
- added LED1: 0805G_(Green), ct-kicad:LED0805-R-RD, F.Cu at (174.8, 65.5)
- added LOGO1: **REF, ct-kicad:awesome-logo, F.Cu at (198.1, 129.8)
- added LOGO2: **REF, ct-kicad:qmk-lite, F.Cu at (207.2, 101.1)
- added LOGO3: **REF, ct-kicad:awesome-logo, B.Cu at (198.1, 129.7)
- added LOGO4: **REF, ct-kicad:qmk-lite, B.Cu at (207.2, 100.6)
- added MOSFET1: AO3401A_C347476, ct-kicad:SOT-23_L2.9-W1.3-P1.90-LS2.4-BR, F.Cu at (164.3, 59.0)
- added PICO1: Pico, rp2040:RPi_Pico_SMD_TH, F.Cu at (145.0, 77.0)
- added PWM1: Conn_01x08_Socket, Connector_JST:JST_EH_S8B-EH_1x08_P2.50mm_Horizontal, F.Cu at (175.2, 145.7)
- added PWR-OUT1: Conn_01x03_Socket, Connector_JST:JST_EH_B3B-EH-A_1x03_P2.50mm_Vertical, F.Cu at (114.5, 24.0)
- added PWR-OUT2: Conn_01x03_Socket, Connector_PinSocket_2.54mm:PinSocket_1x03_P2.54mm_Vertical, F.Cu at (109.4, 24.1)
- added R1: 1206W4F1002T5E, ct-kicad:R1206, F.Cu at (123.8, 91.0)
- added R10: 1206W4F1002T5E, ct-kicad:R1206, F.Cu at (128.2, 120.7)
- added R2: 4D03WGJ0103T5E, ct-kicad:RES-ARRAY-SMD_0603-8P-L3.2-W1.6-BL, F.Cu at (118.3, 107.0)
- added R3: 4D03WGJ0103T5E, ct-kicad:RES-ARRAY-SMD_0603-8P-L3.2-W1.6-BL, F.Cu at (118.3, 92.0)
- added R4: 4D03WGJ0103T5E, ct-kicad:RES-ARRAY-SMD_0603-8P-L3.2-W1.6-BL, F.Cu at (118.3, 87.0)
- added R5: 4D03WGJ0103T5E, ct-kicad:RES-ARRAY-SMD_0603-8P-L3.2-W1.6-BL, F.Cu at (118.3, 72.0)
- added R6: 4.7k, ct-kicad:R1206, F.Cu at (63.1, 131.0)
- added R7: 4.7k, ct-kicad:R1206, F.Cu at (65.6, 131.0)
- added R8: 4.7k, ct-kicad:R1206, F.Cu at (128.2, 117.8)
- added R9: 0402WGF2001TCE, ct-kicad:R0402, F.Cu at (174.6, 67.4)
- added REG-COL1: MC74HC589ADR2G, ct-kicad:SOIC-16_L9.9-W3.9-P1.27-LS6.0-BL, F.Cu at (118.3, 99.5)
- added REG-COL2: MC74HC589ADR2G, ct-kicad:SOIC-16_L9.9-W3.9-P1.27-LS6.0-BL, F.Cu at (118.3, 79.5)
- added REG-ROW1: 74HC595D, ct-kicad:SOIC-16_L9.9-W3.9-P1.27-LS6.0-BL, F.Cu at (118.3, 126.5)
- added REG-ROW2: 74HC595D, ct-kicad:SOIC-16_L9.9-W3.9-P1.27-LS6.0-BL, F.Cu at (118.3, 114.5)
- added RESET1: Conn_01x02_Socket, Connector_JST:JST_EH_B2B-EH-A_1x02_P2.50mm_Vertical, F.Cu at (168.6, 41.0)
- added ROW1: Conn_01x08_Socket, Connector_JST:JST_EH_S8B-EH_1x08_P2.50mm_Horizontal, F.Cu at (67.9, 109.4)
- added ROW2: Conn_01x08_Socket, Connector_JST:JST_EH_S8B-EH_1x08_P2.50mm_Horizontal, F.Cu at (50.4, 105.0)
- added SCREEN1: TYPE-C-31-M-12, ct-kicad:USB-C_SMD-TYPE-C-31-M-12, F.Cu at (110.1, 55.6)
- added SPLIT-USB1: TYPE-C-31-M-12, ct-kicad:USB-C_SMD-TYPE-C-31-M-12, F.Cu at (180.0, 56.0)
- added SPLIT_HAND1: Conn_01x03_Socket, Connector_PinSocket_2.54mm:PinSocket_1x03_P2.54mm_Vertical, F.Cu at (123.0, 53.0)
- added T1: Conn_01x01_Socket, Connector_Pin:Pin_D1.0mm_L10.0mm, F.Cu at (236.4, 118.9)
- added T10: Conn_01x01_Socket, Connector_Pin:Pin_D1.0mm_L10.0mm, F.Cu at (164.7, 71.0)
- added T2: Conn_01x01_Socket, Connector_Pin:Pin_D1.0mm_L10.0mm, F.Cu at (232.7, 118.8)
- added T3: Conn_01x01_Socket, Connector_Pin:Pin_D1.0mm_L10.0mm, F.Cu at (229.4, 118.8)
- added T4: Conn_01x01_Socket, Connector_Pin:Pin_D1.0mm_L10.0mm, F.Cu at (65.5, 147.2)
- added T5: Conn_01x01_Socket, Connector_Pin:Pin_D1.0mm_L10.0mm, F.Cu at (124.9, 100.1)
- added T6: Conn_01x01_Socket, Connector_Pin:Pin_D1.0mm_L10.0mm, F.Cu at (124.9, 104.7)
- added T7: Conn_01x01_Socket, Connector_Pin:Pin_D1.0mm_L10.0mm, F.Cu at (152.8, 34.6)
- added T8: Conn_01x01_Socket, Connector_Pin:Pin_D1.0mm_L10.0mm, F.Cu at (152.8, 29.9)
- added T9: Conn_01x01_Socket, Connector_Pin:Pin_D1.0mm_L10.0mm, F.Cu at (161.3, 71.0)
- added U1: AZC199-04S-MS, ct-kicad:TSOT-23-6_L2.9-W1.6-P0.95-LS2.8-BL, F.Cu at (180.0, 64.3)
- added U10: 8_01A0_008200, ct-kicad:FPC-SMD_8P-P0.50_8.01A0.008200, F.Cu at (175.4, 128.7)
- added U11: 8_01A0_008200, ct-kicad:FPC-SMD_8P-P0.50_8.01A0.008200, F.Cu at (185.4, 128.7)
- added U2: 1N4148W_C81598, ct-kicad:SOD-123F_L2.7-W1.6-LS3.8-RD, F.Cu at (48.1, 130.9)
- added U3: 1N4148W_C81598, ct-kicad:SOD-123F_L2.7-W1.6-LS3.8-RD, F.Cu at (55.6, 130.9)
- added U4: 1N4148W_C81598, ct-kicad:SOD-123F_L2.7-W1.6-LS3.8-RD, F.Cu at (60.7, 130.9)
- added U5: 1N4148W_C81598, ct-kicad:SOD-123F_L2.7-W1.6-LS3.8-RD, F.Cu at (53.1, 130.9)
- added U6: 1N4148W_C81598, ct-kicad:SOD-123F_L2.7-W1.6-LS3.8-RD, F.Cu at (58.0, 130.9)
- added U9: 8_01A0_008200, ct-kicad:FPC-SMD_8P-P0.50_8.01A0.008200, F.Cu at (165.4, 128.7)
- added VCC_BYPASS1: Conn_01x03_Socket, Connector_PinSocket_2.54mm:PinSocket_1x03_P2.54mm_Vertical, F.Cu at (167.7, 52.9)
Other:
- board outline added: 130 x 85 mm
