File: mk19-pcb.kicad_pcb (KiCad board)
At the start: 2 copper layers, 130 x 85 mm, 88 parts, among them J1 Conn_01x02_Socket, J10 Conn_01x02_Socket, J11 Conn_01x02_Socket, J2 Conn_01x02_Socket, J4 Conn_01x02_Socket, J7 Conn_01x02_Socket, J9 Conn_01x02_Socket, T1 Conn_01x01_Socket, T10 Conn_01x01_Socket, U1 AZC199-04S-MS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

Commit message: adding jumper for clk pulldown
Parts:
- added CLK_PULL1: Conn_01x02_Socket, Connector_PinSocket_2.54mm:PinSocket_1x02_P2.54mm_Vertical, F.Cu at (128.0, 83.9)
- added R11: 1206W4F1002T5E, ct-kicad:R1206, F.Cu at (116.2, 53.6)
- moved R8 4.89 mm to (128.0, 79.5)
Connections:
- R8 pad 1: SPI1_CLK -> Net-(CLK_PULL1-Pin_1)
- SPLIT_HAND1 pad 3: +3V3 -> Net-(SPLIT_HAND1-Pin_3)
Routing:
- net GND: track 622.0 -> 641.5 mm, vias 136 -> 137
- net Net-(SPLIT_HAND1-Pin_3): track 0.00 -> 6.95 mm
- net Net-(CLK_PULL1-Pin_1): track 0.00 -> 2.90 mm
- net +3V3: track 359.6 -> 362.3 mm
- net SPI1_CLK: track 198.1 -> 198.5 mm, vias 16 -> 15
Other:
- board text added: "CLK-PULL"

Commit message: production files
Parts:
- moved C6 0.99 mm to (167.0, 69.4), turned to 0 degrees
Routing:
- net GND: track 641.5 -> 688.5 mm
- net VCC: track 276.7 -> 284.7 mm, vias 4 -> 5
- net +3V3: track 362.3 -> 366.8 mm
- net LED_DI_3v3: track 9.96 -> 10.6 mm
