File: mk19-pcb.kicad_sch (KiCad schematic)
At the start: 103 parts, among them J1 Conn_01x02_Socket, J10 Conn_01x02_Socket, J11 Conn_01x02_Socket, J2 Conn_01x02_Socket, J4 Conn_01x02_Socket, J7 Conn_01x02_Socket, J9 Conn_01x02_Socket, P1 FH26W-13S-0_3SHW(60), P10 FH26W-13S-0_3SHW(60), P11 FH26W-13S-0_3SHW(60), P2 FH26W-13S-0_3SHW(60), P3 FH26W-13S-0_3SHW(60), P4 FH26W-13S-0_3SHW(60), P5 FH26W-13S-0_3SHW(60), P6 FH26W-13S-0_3SHW(60), P7 FH26W-13S-0_3SHW(60), P8 FH26W-13S-0_3SHW(60), P9 FH26W-13S-0_3SHW(60), T1 Conn_01x01_Socket, T10 Conn_01x01_Socket, U1 AZC199-04S-MS, U10 8_01A0_008200, U11 8_01A0_008200, U2 1N4148W_C81598, U3 1N4148W_C81598, U4 1N4148W_C81598, U5 1N4148W_C81598, U6 1N4148W_C81598, U7 HC-FPC-05-10-16RLTAG, U8 ECT818001569, U9 8_01A0_008200

Commit message: production files
Parts:
- CLK_PULL1: renamed from CLK_PULL; now left out of the parts list
- COL_JOIN1, COL_JOIN2, J1, J10, J11, J2, J4, J7, J9, MISO_PULL1, SPLIT_HAND1, VCC_BYPASS1: now left out of the parts list
- CYBOARD-MACRO1: LCSC C2914211 -> C5213735
Changed lines of the file:
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@@
     (stroke (width 0) (type default))
   )
-  (wire (pts (xy 254 67.31) (xy 274.32 67.31))
-    (stroke (width 0) (type default))
-  )
   (wire (pts (xy 650.24 111.76) (xy 650.24 113.03))
     (stroke (width 0) (type default))
@@
     (stroke (width 0) (type default))
   )
+  (wire (pts (xy 254 67.31) (xy 274.32 67.31))
+    (stroke (width 0) (type default))
+  )
   (wire (pts (xy 654.05 74.93) (xy 652.78 74.93))
     (stroke (width 0) (type default))
@@
   )
   (symbol (lib_id "Connector:Conn_01x02_Socket") (at 245.11 200.66 0) (unit 1)
-    (in_bom yes) (on_board yes) (dnp no) (fields_autoplaced)
+    (in_bom no) (on_board yes) (dnp no) (fields_autoplaced)
     (property "Reference" "COL_JOIN1" (at 246.38 200.66 0)
       (effects (font (size 1.27 1.27)) (justify left))
@@
   )
   (symbol (lib_id "Connector:Conn_01x03_Socket") (at 316.23 44.45 180) (unit 1)
-    (in_bom yes) (on_board yes) (dnp no) (fields_autoplaced)
+    (in_bom no) (on_board yes) (dnp no) (fields_autoplaced)
     (property "Reference" "SPLIT_HAND1" (at 316.865 36.83 0)
       (effects (font (size 1.27 1.27)))
@@
   )
   (symbol (lib_id "Connector:Conn_01x03_Socket") (at 154.94 236.22 90) (unit 1)
-    (in_bom yes) (on_board yes) (dnp no) (fields_autoplaced)
+    (in_bom no) (on_board yes) (dnp no) (fields_autoplaced)
     (property "Reference" "VCC_BYPASS1" (at 154.94 231.14 90)
       (effects (font (size 1.27 1.27)))
@@
   )
   (symbol (lib_id "Connector:Conn_01x02_Socket") (at 425.45 342.9 90) (unit 1)
-    (in_bom yes) (on_board yes) (dnp no) (fields_autoplaced)
+    (in_bom no) (on_board yes) (dnp no) (fields_autoplaced)
     (property "Reference" "J9" (at 433.07 343.535 0)
       (effects (font (size 1.27 1.27)) hide)
@@
   )
   (symbol (lib_id "Connector:Conn_01x02_Socket") (at 157.48 210.82 270) (unit 1)
-    (in_bom yes) (on_board yes) (dnp no) (fields_autoplaced)
+    (in_bom no) (on_board yes) (dnp no) (fields_autoplaced)
     (property "Reference" "COL_JOIN2" (at 158.75 208.915 90)
       (effects (font (size 1.27 1.27)) (justify left))
@@
   )
   (symbol (lib_id "Connector:Conn_01x02_Socket") (at 375.92 342.9 90) (unit 1)
-    (in_bom yes) (on_board yes) (dnp no) (fields_autoplaced)
+    (in_bom no) (on_board yes) (dnp no) (fields_autoplaced)
     (property "Reference" "J4" (at 383.54 343.535 0)
       (effects (font (size 1.27 1.27)) hide)
@@
   )
   (symbol (lib_id "Connector:Conn_01x02_Socket") (at 412.75 205.74 180) (unit 1)
-    (in_bom yes) (on_board yes) (dnp no) (fields_autoplaced)
+    (in_bom no) (on_board yes) (dnp no) (fields_autoplaced)
     (property "Reference" "J7" (at 413.385 198.12 0)
       (effects (font (size 1.27 1.27)))
@@
   )
   (symbol (lib_id "Connector:Conn_01x02_Socket") (at 307.34 87.63 180) (unit 1)
-    (in_bom yes) (on_board yes) (dnp no) (fields_autoplaced)
-    (property "Reference" "CLK_PULL" (at 307.975 80.01 0)
+    (in_bom no) (on_board yes) (dnp no) (fields_autoplaced)
+    (property "Reference" "CLK_PULL1" (at 307.975 80.01 0)
       (effects (font (size 1.27 1.27)))
     )
@@
       (project "mk19-pcb"
         (path "/2353ceae-84c1-4f16-856e-bae2658fe2c9"
-          (reference "CLK_PULL") (unit 1)
+          (reference "CLK_PULL1") (unit 1)
         )
       )
@@
   )
   (symbol (lib_id "Connector:Conn_01x02_Socket") (at 452.12 205.74 180) (unit 1)
-    (in_bom yes) (on_board yes) (dnp no) (fields_autoplaced)
+    (in_bom no) (on_board yes) (dnp no) (fields_autoplaced)
     (property "Reference" "J1" (at 452.755 198.12 0)
       (effects (font (size 1.27 1.27)))
@@
   )
   (symbol (lib_id "Connector:Conn_01x02_Socket") (at 332.74 342.9 90) (unit 1)
-    (in_bom yes) (on_board yes) (dnp no) (fields_autoplaced)
+    (in_bom no) (on_board yes) (dnp no) (fields_autoplaced)
     (property "Reference" "J10" (at 340.36 343.535 0)
       (effects (font (size 1.27 1.27)) hide)
@@
       (effects (font (size 1.27 1.27)) (justify left) hide)
     )
-    (property "LCSC" "C2914211" (at 246.38 62.23 0)
+    (property "LCSC" "C5213735" (at 246.38 62.23 0)
       (effects (font (size 1.27 1.27)) hide)
     )
@@
   )
   (symbol (lib_id "Connector:Conn_01x02_Socket") (at 422.91 284.48 180) (unit 1)
-    (in_bom yes) (on_board yes) (dnp no) (fields_autoplaced)
+    (in_bom no) (on_board yes) (dnp no) (fields_autoplaced)
     (property "Reference" "J11" (at 423.545 276.86 0)
       (effects (font (size 1.27 1.27)) hide)
@@
   )
   (symbol (lib_id "Connector:Conn_01x02_Socket") (at 491.49 205.74 180) (unit 1)
-    (in_bom yes) (on_board yes) (dnp no) (fields_autoplaced)
+    (in_bom no) (on_board yes) (dnp no) (fields_autoplaced)
     (property "Reference" "J2" (at 492.125 198.12 0)
       (effects (font (size 1.27 1.27)))
@@
   )
   (symbol (lib_id "Connector:Conn_01x02_Socket") (at 322.58 95.25 180) (unit 1)
-    (in_bom yes) (on_board yes) (dnp no) (fields_autoplaced)
+    (in_bom no) (on_board yes) (dnp no) (fields_autoplaced)
     (property "Reference" "MISO_PULL1" (at 323.215 87.63 0)
       (effects (font (size 1.27 1.27)))
