File: mk19-pcb.kicad_sch (KiCad schematic)
At the start: 103 parts, among them J1 Conn_01x02_Socket, J10 Conn_01x02_Socket, J11 Conn_01x02_Socket, J2 Conn_01x02_Socket, J4 Conn_01x02_Socket, J7 Conn_01x02_Socket, J9 Conn_01x02_Socket, P1 FH26W-13S-0_3SHW(60), P10 FH26W-13S-0_3SHW(60), P11 FH26W-13S-0_3SHW(60)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

Commit message: working on improving the readme
Other:
- note added: "Rows and Columns"
- moved on the sheet: ADC1, AUDIO1, C2, C4, C5, C6, C7, C8, C9, CLK_PULL1, COL_CS_MOS1, COL_JOIN1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
